Commit message: Lidar can be used

File: src/medibot/medibot/medibot_description/urdf/medibot_medibotv4.urdf (robot description, URDF)
Before this commit: robot medibot_medibotv4, 25 links, 24 joints
Links:
- removed link left_wheel
- removed link right_wheel
- removed link sonar
- added link wheel_left_link, mass 2.266879326854612; collision mesh filename=package://medibot_description/meshes/meshes/left_wheel.stl scale=0.001 0.001 0.001; visual mesh filename=package://medibot_description/meshes/meshes/left_wheel.stl scale=0.001 0.001 0.001
- added link wheel_right_link, mass 2.266879326854595; collision mesh filename=package://medibot_description/meshes/meshes/right_wheel.stl scale=0.001 0.001 0.001; visual mesh filename=package://medibot_description/meshes/meshes/right_wheel.stl scale=0.001 0.001 0.001
Joints:
- removed joint left_wheel_joint
- removed joint right_wheel_joint
- removed joint sonar_joint
- added joint wheel_left_joint: type continuous, parent left_motor, child wheel_left_link, origin xyz=0.036 0.1255 -0.0545 rpy=0 0 0, axis -0.0 1.0 0.0
- added joint wheel_right_joint: type continuous, parent right_motor, child wheel_right_link, origin xyz=0.036 -0.1255 -0.0545 rpy=0 0 0, axis -0.0 1.0 0.0
- joint pan_servo_joint: type continuous -> fixed
- joint tilt_servo_joint: type continuous -> fixed

File: src/medibot/medibot_simulations/medibot_gazebo/urdf/medibot_medibotv4.urdf (robot description, URDF)
Before this commit: robot medibot_medibotv4, 23 links, 22 joints
Links:
- removed link lidar
- added link base_footprint
- added link base_scan, mass 0.052814160089970474; collision mesh filename=package://medibot_gazebo/models/medibot_common/meshes/lidar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 scale=0.001 0.001 0.001; visual mesh filename=package://medibot_gazebo/models/medibot_common/meshes/lidar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 scale=0.001 0.001 0.001
Joints:
- added joint base_joint: type fixed, parent base_footprint, child base_link, origin xyz=0.0 0.0 0.010 rpy=0 0 0
- joint lidar_joint: child lidar -> base_scan
