Commit message: 10/12/24

File: src/medibot/medibot_simulations/medibot_gazebo/urdf/medibot_medibotv4.urdf (robot description, URDF)
Before this commit: robot medibot_medibotv4, 25 links, 24 joints
Links:
- link base_link: geometry collision mesh filename=package://medibot_gazebo/models/medibot_common/meshes/base_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 scale=0.001 0.001 0.001; visual mesh filename=package://medibot_gazebo/models/medibot_common/meshes/base_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 scale=0.001 0.001 0.001
- link body: geometry collision mesh filename=package://medibot_gazebo/models/medibot_common/meshes/body.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 scale=0.001 0.001 0.001; visual mesh filename=package://medibot_gazebo/models/medibot_common/meshes/body.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 scale=0.001 0.001 0.001
- link bottom_panel: geometry collision mesh filename=package://medibot_gazebo/models/medibot_common/meshes/botto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 scale=0.001 0.001 0.001; visual mesh filename=package://medibot_gazebo/models/medibot_common/meshes/botto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 scale=0.001 0.001 0.001
- link camera: geometry collision mesh filename=package://medibot_gazebo/models/medibot_common/meshes/camer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 scale=0.001 0.001 0.001; visual mesh filename=package://medibot_gazebo/models/medibot_common/meshes/camer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 scale=0.001 0.001 0.001
- link camera_housing: geometry collision mesh filename=package://medibot_gazebo/models/medibot_common/meshes/camer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 scale=0.001 0.001 0.001; visual mesh filename=package://medibot_gazebo/models/medibot_common/meshes/camer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 scale=0.001 0.001 0.001
- link caster: geometry collision mesh filename=package://medibot_gazebo/models/medibot_common/meshes/caste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 scale=0.001 0.001 0.001; visual mesh filename=package://medibot_gazebo/models/medibot_common/meshes/caste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 scale=0.001 0.001 0.001
- link circuit_housing: geometry collision mesh filename=package://medibot_gazebo/models/medibot_common/meshes/circu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 scale=0.001 0.001 0.001; visual mesh filename=package://medibot_gazebo/models/medibot_common/meshes/circu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 scale=0.001 0.001 0.001
- link circuit_panel: geometry collision mesh filename=package://medibot_gazebo/models/medibot_common/meshes/circu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 scale=0.001 0.001 0.001; visual mesh filename=package://medibot_gazebo/models/medibot_common/meshes/circu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 scale=0.001 0.001 0.001
- link left_motor: geometry collision mesh filename=package://medibot_gazebo/models/medibot_common/meshes/left_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 scale=0.001 0.001 0.001; visual mesh filename=package://medibot_gazebo/models/medibot_common/meshes/left_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 scale=0.001 0.001 0.001
- link left_realsense: geometry collision mesh filename=package://medibot_gazebo/models/medibot_common/meshes/left_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 scale=0.001 0.001 0.001; visual mesh filename=package://medibot_gazebo/models/medibot_common/meshes/left_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 scale=0.001 0.001 0.001
- link left_wheel: geometry collision mesh filename=package://medibot_gazebo/models/medibot_common/meshes/left_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 scale=0.001 0.001 0.001; visual mesh filename=package://medibot_gazebo/models/medibot_common/meshes/left_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 scale=0.001 0.001 0.001
- link lidar: geometry collision mesh filename=package://medibot_gazebo/models/medibot_common/meshes/lidar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 scale=0.001 0.001 0.001; visual mesh filename=package://medibot_gazebo/models/medibot_common/meshes/lidar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 scale=0.001 0.001 0.001
- link monitor: geometry collision mesh filename=package://medibot_gazebo/models/medibot_common/meshes/monit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 scale=0.001 0.001 0.001; visual mesh filename=package://medibot_gazebo/models/medibot_common/meshes/monit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 scale=0.001 0.001 0.001
- link mount: geometry collision mesh filename=package://medibot_gazebo/models/medibot_common/meshes/mount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 scale=0.001 0.001 0.001; visual mesh filename=package://medibot_gazebo/models/medibot_common/meshes/mount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 scale=0.001 0.001 0.001
- link pan_servo: geometry collision mesh filename=package://medibot_gazebo/models/medibot_common/meshes/pan_s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 scale=0.001 0.001 0.001; visual mesh filename=package://medibot_gazebo/models/medibot_common/meshes/pan_s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 scale=0.001 0.001 0.001
- link pan_tilt_mount: geometry collision mesh filename=package://medibot_gazebo/models/medibot_common/meshes/pan_t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 scale=0.001 0.001 0.001; visual mesh filename=package://medibot_gazebo/models/medibot_common/meshes/pan_t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 scale=0.001 0.001 0.001
- link realsense_housing: geometry collision mesh filename=package://medibot_gazebo/models/medibot_common/meshes/reals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 scale=0.001 0.001 0.001; visual mesh filename=package://medibot_gazebo/models/medibot_common/meshes/reals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 scale=0.001 0.001 0.001
- link right_motor: geometry collision mesh filename=package://medibot_gazebo/models/medibot_common/meshes/right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 scale=0.001 0.001 0.001; visual mesh filename=package://medibot_gazebo/models/medibot_common/meshes/right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 scale=0.001 0.001 0.001
- link right_realsense: geometry collision mesh filename=package://medibot_gazebo/models/medibot_common/meshes/right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 scale=0.001 0.001 0.001; visual mesh filename=package://medibot_gazebo/models/medibot_common/meshes/right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 scale=0.001 0.001 0.001
- link right_wheel: geometry collision mesh filename=package://medibot_gazebo/models/medibot_common/meshes/right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 scale=0.001 0.001 0.001; visual mesh filename=package://medibot_gazebo/models/medibot_common/meshes/right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 scale=0.001 0.001 0.001
- link sonar: geometry collision mesh filename=package://medibot_gazebo/models/medibot_common/meshes/sonar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 scale=0.001 0.001 0.001; visual mesh filename=package://medibot_gazebo/models/medibot_common/meshes/sonar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 scale=0.001 0.001 0.001
- link stand: geometry collision mesh filename=package://medibot_gazebo/models/medibot_common/meshes/stand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 scale=0.001 0.001 0.001; visual mesh filename=package://medibot_gazebo/models/medibot_common/meshes/stand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 scale=0.001 0.001 0.001
- link tilt_servo: geometry collision mesh filename=package://medibot_gazebo/models/medibot_common/meshes/tilt_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 scale=0.001 0.001 0.001; visual mesh filename=package://medibot_gazebo/models/medibot_common/meshes/tilt_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 scale=0.001 0.001 0.001
- link top_panel: geometry collision mesh filename=package://medibot_gazebo/models/medibot_common/meshes/top_p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 scale=0.001 0.001 0.001; visual mesh filename=package://medibot_gazebo/models/medibot_common/meshes/top_p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 scale=0.001 0.001 0.001

Commit message: medibot move

File: src/medibot/medibot_simulations/medibot_gazebo/urdf/medibot_medibotv4.urdf (robot description, URDF)
Before this commit: robot medibot_medibotv4, 24 links, 23 joints
Joints:
- joint wheel_left_joint: limit (none) -> effort=1000 velocity=1000
- joint wheel_right_joint: limit (none) -> effort=1000 velocity=1000
