Commit message: edited urdf

File: src/medibot/medibot_simulations/medibot_gazebo/urdf/medibot_medibotv5.urdf (robot description, URDF)
Before this commit: robot medibot_medibotv4, 23 links, 22 joints
Links:
- removed link wheel_left_link
- removed link wheel_right_link
- added link base_footprint
- added link left_wheel, mass 2.266879326854612; collision mesh filename=package://medibot_gazebo/models/medibot_common/meshes/left_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 scale=0.001 0.001 0.001; visual mesh filename=package://medibot_gazebo/models/medibot_common/meshes/left_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 scale=0.001 0.001 0.001
- added link right_wheel, mass 2.266879326854595; collision mesh filename=package://medibot_gazebo/models/medibot_common/meshes/right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 scale=0.001 0.001 0.001; visual mesh filename=package://medibot_gazebo/models/medibot_common/meshes/right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 scale=0.001 0.001 0.001
- added link sonar, mass 2.6048925401122753; collision mesh filename=package://medibot_gazebo/models/medibot_common/meshes/sonar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 scale=0.001 0.001 0.001; visual mesh filename=package://medibot_gazebo/models/medibot_common/meshes/sonar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 scale=0.001 0.001 0.001
Joints:
- removed joint wheel_right_joint
- added joint base_joint: type fixed, parent base_footprint, child base_link, origin xyz=0.0 0.0 0.010 rpy=0 0 0
- added joint right_joint: type continuous, parent right_motor, child right_wheel, origin xyz=0.036 -0.1255 -0.0545 rpy=0 0 0, axis -0.0 1.0 0.0
- added joint sonar_joint: type fixed, parent stand, child sonar, origin xyz=0.0 0.0 0.625 rpy=0 0 0
- joint pan_servo_joint: type fixed -> continuous
- joint tilt_servo_joint: type fixed -> continuous
- joint wheel_left_joint: child wheel_left_link -> left_wheel

Commit message: mapping

File: src/medibot/medibot_simulations/medibot_gazebo/urdf/medibot_medibotv5.urdf (robot description, URDF)
Before this commit: robot medibot_medibotv5, 25 links, 24 joints
Links:
- removed link left_wheel
- removed link lidar
- removed link right_wheel
- removed link sonar
- added link base_scan, mass 0.052814160089970474; collision mesh filename=package://medibot_gazebo/models/medibot_common/meshes/lidar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 scale=0.001 0.001 0.001; visual mesh filename=package://medibot_gazebo/models/medibot_common/meshes/lidar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 scale=0.001 0.001 0.001
- added link wheel_left_link, mass 2.266879326854612; collision mesh filename=package://medibot_gazebo/models/medibot_common/meshes/left_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 scale=0.001 0.001 0.001; visual mesh filename=package://medibot_gazebo/models/medibot_common/meshes/left_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 scale=0.001 0.001 0.001
- added link wheel_right_link, mass 2.266879326854595; collision mesh filename=package://medibot_gazebo/models/medibot_common/meshes/right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 scale=0.001 0.001 0.001; visual mesh filename=package://medibot_gazebo/models/medibot_common/meshes/right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 scale=0.001 0.001 0.001
Joints:
- removed joint right_joint
- removed joint sonar_joint
- added joint wheel_right_joint: type continuous, parent right_motor, child wheel_right_link, origin xyz=0.036 -0.1255 -0.0545 rpy=0 0 0, axis -0.0 1.0 0.0, limit effort=1000 velocity=1000
- joint lidar_joint: child lidar -> base_scan
- joint pan_servo_joint: type continuous -> fixed
- joint tilt_servo_joint: type continuous -> fixed
- joint wheel_left_joint: child left_wheel -> wheel_left_link; limit (none) -> effort=1000 velocity=1000
